Commit message: refactor: rename project to autonomous mobile robot

File: src/autonomous_mobile_robot_description/urdf/autonomous_mobile_robot.xacro (robot description, xacro)
@@ -1,6 +1,6 @@
 <?xml version="1.0"?>
-<robot xmlns:xacro="http://www.ros.org/wiki/xacro" name="marpy">
-  <xacro:include filename="$(find marpy_description)/urdf/materials.xacro" />
-  <xacro:include filename="$(find marpy_description)/urdf/marpy_gazebo.xacro" />
+<robot xmlns:xacro="http://www.ros.org/wiki/xacro" name="autonomous_mobile_robot">
+  <xacro:include filename="$(find autonomous_mobile_robot_description)/urdf/materials.xacro" />
+  <xacro:include filename="$(find autonomous_mobile_robot_description)/urdf/autonomous_mobile_robot_gazebo.xacro" />
   <!-- ==================== Properties ==================== -->
   <!-- Wheel geometry (from CLAUDE.md specs) -->
@@ -28,5 +28,5 @@
       <origin xyz="0 0 0" rpy="0 0 0" />
       <geometry>
-        <mesh filename="package://marpy_description/meshes/base_link.STL" />
+        <mesh filename="package://autonomous_mobile_robot_description/meshes/base_link.STL" />
       </geometry>
       <material name="light_blue" />
@@ -35,5 +35,5 @@
       <origin xyz="0 0 0" rpy="0 0 0" />
       <geometry>
-        <mesh filename="package://marpy_description/meshes/base_link.STL" />
+        <mesh filename="package://autonomous_mobile_robot_description/meshes/base_link.STL" />
       </geometry>
     </collision>
@@ -52,5 +52,5 @@
       <origin xyz="0 0 0" rpy="0 0 0" />
       <geometry>
-        <mesh filename="package://marpy_description/meshes/imu_link.STL" />
+        <mesh filename="package://autonomous_mobile_robot_description/meshes/imu_link.STL" />
       </geometry>
       <material name="dark_grey" />
@@ -59,5 +59,5 @@
       <origin xyz="0 0 0" rpy="0 0 0" />
       <geometry>
-        <mesh filename="package://marpy_description/meshes/imu_link.STL" />
+        <mesh filename="package://autonomous_mobile_robot_description/meshes/imu_link.STL" />
       </geometry>
     </collision>
@@ -81,5 +81,5 @@
       <origin xyz="0 0 0" rpy="0 0 0" />
       <geometry>
-        <mesh filename="package://marpy_description/meshes/left_wheel.STL" />
+        <mesh filename="package://autonomous_mobile_robot_description/meshes/left_wheel.STL" />
       </geometry>
       <material name="dark_grey" />
@@ -113,5 +113,5 @@
       <origin xyz="0 0 0" rpy="0 0 0" />
       <geometry>
-        <mesh filename="package://marpy_description/meshes/right_wheel.STL" />
+        <mesh filename="package://autonomous_mobile_robot_description/meshes/right_wheel.STL" />
       </geometry>
       <material name="dark_grey" />
@@ -145,5 +145,5 @@
       <origin xyz="0 0 0" rpy="0 0 0" />
       <geometry>
-        <mesh filename="package://marpy_description/meshes/caster_wheel.STL" />
+        <mesh filename="package://autonomous_mobile_robot_description/meshes/caster_wheel.STL" />
       </geometry>
       <material name="dark_grey" />

File: src/autonomous_mobile_robot_description/urdf/autonomous_mobile_robot_gazebo.xacro (robot description, xacro)
@@ -86,5 +86,5 @@
   <!--
     DiffDrive plugin: subscribes to /cmd_vel and drives the wheel joints.
-    Odometry is NOT computed here - marpy_localization handles it from
+    Odometry is NOT computed here - autonomous_mobile_robot_localization handles it from
     /joint_states, keeping the sim pipeline identical to real hardware.
   -->

Commit message: Add Gazebo house camera and collision reset support

File: src/autonomous_mobile_robot_description/urdf/autonomous_mobile_robot.xacro (robot description, xacro)
@@ -3,4 +3,5 @@
   <xacro:include filename="$(find autonomous_mobile_robot_description)/urdf/materials.xacro" />
   <xacro:include filename="$(find autonomous_mobile_robot_description)/urdf/autonomous_mobile_robot_gazebo.xacro" />
+  <xacro:include filename="$(find autonomous_mobile_robot_description)/urdf/camera.xacro" />
   <!-- ==================== Properties ==================== -->
   <!-- Wheel geometry for the differential-drive base. -->
@@ -32,9 +33,8 @@
       <material name="light_blue" />
     </visual>
-    <collision>
-      <origin xyz="0 0 0" rpy="0 0 0" />
-      <geometry>
-        <mesh filename="package://autonomous_mobile_robot_description/meshes/base_link.STL" />
-      </geometry>
+    <collision name="base_collision">
+      <!-- Padded chassis and wheel envelope; box works with Gazebo DART physics. -->
+      <origin xyz="-0.02015 0 0.02723" rpy="0 0 0" />
+      <geometry><box size="0.22 0.16 0.11" /></geometry>
     </collision>
   </link>

File: src/autonomous_mobile_robot_description/urdf/autonomous_mobile_robot_gazebo.xacro (robot description, xacro)
@@ -84,4 +84,16 @@
     </sensor>
   </gazebo>
+  <!-- Contact reporting for the simulation reset controller. -->
+  <gazebo reference="base_link">
+    <sensor name="base_contact" type="contact">
+      <always_on>true</always_on>
+      <update_rate>30</update_rate>
+      <contact>
+        <collision>base_footprint_fixed_joint_lump__base_collision_collision</collision>
+        <!-- Contact topics are configured inside <contact> for Gazebo Sensors. -->
+        <topic>/robot/contacts</topic>
+      </contact>
+    </sensor>
+  </gazebo>
   <!--
     DiffDrive plugin: subscribes to /cmd_vel and drives the wheel joints.
